Commit message: add: new meshes, etc

File: urdf/seekurjr_without_controller.urdf (robot description, URDF)
Before this commit: robot seekurjr, 9 links, 8 joints
Links:
- link back_left_wheel: geometry collision mesh filename=package://seekurjr_gazebo/meshes/seekurjr_wheel_bl.stl; visual mesh filename=package://seekurjr_gazebo/meshes/seekurjr_wheel_bl.stl
- link back_right_wheel: geometry collision mesh filename=package://seekurjr_gazebo/meshes/seekurjr_wheel_br.stl; visual mesh filename=package://seekurjr_gazebo/meshes/seekurjr_wheel_br.stl
- link base_link: geometry collision mesh filename=package://seekurjr_gazebo/meshes/seekurjr_body_new_low.stl; visual mesh filename=package://seekurjr_gazebo/meshes/seekurjr_body_new_low.stl
- link front_left_wheel: geometry collision mesh filename=package://seekurjr_gazebo/meshes/seekurjr_wheel_fl.stl; visual mesh filename=package://seekurjr_gazebo/meshes/seekurjr_wheel_fl.stl
- link front_right_wheel: geometry collision mesh filename=package://seekurjr_gazebo/meshes/seekurjr_wheel_fr.stl; visual mesh filename=package://seekurjr_gazebo/meshes/seekurjr_wheel_fr.stl
- link hokuyo_laser_link: geometry visual mesh filename=package://seekurjr_gazebo/meshes/seekurjr_lms1xx_low.stl scale=0.5 0.5 0.5
