Commit message: add: full model, fixed wheels, dae for body

File: urdf/seekurjr.urdf (robot description, URDF)
Before this commit: robot seekurjr, 5 links, 4 joints
Links:
- added link bl_wheel; collision mesh filename=package://seekurjr_gazebo/meshes/seekurjr_left_side_wheel_l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 scale=1 1 1; visual mesh filename=package://seekurjr_gazebo/meshes/seekurjr_left_side_wheel_l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 scale=1 1 1
- added link br_wheel; collision mesh filename=package://seekurjr_gazebo/meshes/seekurjr_right_side_wheel_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 scale=1 1 1; visual mesh filename=package://seekurjr_gazebo/meshes/seekurjr_right_side_wheel_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 scale=1 1 1
- added link fl_wheel; collision mesh filename=package://seekurjr_gazebo/meshes/seekurjr_left_side_wheel_l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 scale=1 1 1; visual mesh filename=package://seekurjr_gazebo/meshes/seekurjr_left_side_wheel_l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 scale=1 1 1
- added link fr_wheel; collision mesh filename=package://seekurjr_gazebo/meshes/seekurjr_right_side_wheel_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 scale=1 1 1; visual mesh filename=package://seekurjr_gazebo/meshes/seekurjr_right_side_wheel_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 scale=1 1 1
- link base_link: geometry collision mesh filename=package://seekurjr_gazebo/meshes/seekurjr_body_new_low2.stl scale=1 1 1; visual mesh filename=package://seekurjr_gazebo/meshes/seekurjr_body_new_low2.dae scale=1 1 1
Joints:
- added joint bl_wheel_joint: type fixed, parent base_link, child bl_wheel, origin xyz=-0.215 0.32 0.083 rpy=0 0 0
- added joint br_wheel_joint: type fixed, parent base_link, child br_wheel, origin xyz=-0.215 -0.32 0.083 rpy=0 0 0
- added joint fl_wheel_joint: type fixed, parent base_link, child fl_wheel, origin xyz=0.215 0.32 0.083 rpy=0 0 0
- added joint fr_wheel_joint: type fixed, parent base_link, child fr_wheel, origin xyz=0.215 -0.32 0.083 rpy=0 0 0, limit lower=-100 upper=100 effort=30 velocity=1.0

Commit message: add: wheels working, changes in inertial tensors for most links

File: urdf/seekurjr.urdf (robot description, URDF)
Before this commit: robot seekurjr, 9 links, 8 joints
Links:
- link base_link: mass 77.0 -> 70.0
- link bl_wheel: mass None -> 1.75
- link br_wheel: mass None -> 1.75
- link fl_wheel: mass None -> 1.75
- link fr_wheel: mass None -> 1.75
Joints:
- joint bl_wheel_joint: axis (none) -> 0 1 0; limit (none) -> lower=-100 upper=100 effort=30 velocity=1.0; type fixed -> revolute
- joint br_wheel_joint: axis (none) -> 0 1 0; limit (none) -> lower=-100 upper=100 effort=30 velocity=1.0; type fixed -> revolute
- joint fl_wheel_joint: axis (none) -> 0 1 0; limit (none) -> lower=-100 upper=100 effort=30 velocity=1.0; type fixed -> revolute
- joint fr_wheel_joint: axis (none) -> 0 1 0; type fixed -> revolute
